Commit message: 6.4.2 tbc

File: study/chapt6/chapt6_ws/src/fishbot_description/urdf/fishbot/base.urdf.xacro (robot description, xacro)
@@ -1,6 +1,14 @@
 <?xml version="1.0"?>
 <robot xmlns:xacro="http://www.ros.org/wiki/xacro">
+    <!-- 包含惯性宏定义 -->
+    <xacro:include filename="$(find fishbot_description)/urdf/fishbot/common_inertia.xacro" />
     <!-- 机器人底座 -->
     <xacro:macro name="base_xacro" params="length radius">
+        <link name="base_footprint" />
+        <joint name="base_joint" type="fixed">
+            <parent link="base_footprint"/>
+            <child link="base_link"/>
+            <origin xyz="0 0 ${length/2.0+0.032-0.001}" rpy="0 0 0" />
+        </joint>
         <link name="base_link">
             <visual>
@@ -13,4 +21,11 @@
                 </material>
             </visual>
+            <collision>
+                <origin xyz="0 0 0" rpy="0 0 0"/>
+                <geometry>
+                    <cylinder length="${length}" radius="${radius}" />
+                </geometry>
+            </collision>
+            <xacro:cylinder_inertia m="1.0" r="${radius}" h="${length}" />
         </link>
     </xacro:macro>

File: study/chapt6/chapt6_ws/src/fishbot_description/urdf/fishbot/fishbot.urdf.xacro (robot description, xacro)
@@ -1,4 +1,5 @@
 <?xml version="1.0"?>
-<robot xmlns:xacro="http://www.ros.org/wiki/xacro">
+<robot xmlns:xacro="http://www.ros.org/wiki/xacro" name="fishbot">
+    <!-- 包含基座宏定义 -->
     <xacro:include filename="$(find fishbot_description)/urdf/fishbot/base.urdf.xacro" />
     <!-- 包含传感器宏定义 -->
@@ -6,5 +7,8 @@
     <xacro:include filename="$(find fishbot_description)/urdf/fishbot/sensor/camera.urdf.xacro" />
     <xacro:include filename="$(find fishbot_description)/urdf/fishbot/sensor/laser.urdf.xacro" />
-    <!-- 定义机器人 -->
+    <!-- 包含轮子宏定义 -->
+    <xacro:include filename="$(find fishbot_description)/urdf/fishbot/actuator/wheel.urdf.xacro" />
+    <xacro:include filename="$(find fishbot_description)/urdf/fishbot/actuator/caster.urdf.xacro" />
+    <!-- 基座 -->
     <xacro:base_xacro length="0.12" radius="0.1" />
     <!-- 传感器 -->
@@ -12,3 +16,8 @@
     <xacro:camera_xacro xyz="0.1 0 0.075" />
     <xacro:laser_xacro xyz="0 0 0.1" />
+    <!-- 轮子 -->
+    <xacro:wheel_xacro wheel_name="left_wheel" xyz="0 0.10 -0.06" />
+    <xacro:wheel_xacro wheel_name="right_wheel" xyz="0 -0.10 -0.06" />
+    <xacro:caster_xacro caster_name="front_caster" xyz="0.08 0.0 -0.076" />
+    <xacro:caster_xacro caster_name="back_caster" xyz="-0.08 0.0 -0.076" />
 </robot>

File: study/chapt6/chapt6_ws/src/fishbot_description/urdf/fishbot/sensor/camera.urdf.xacro (robot description, xacro)
@@ -1,4 +1,5 @@
 <?xml version="1.0"?>
 <robot xmlns:xacro="http://www.ros.org/wiki/xacro">
+    <xacro:include filename="$(find fishbot_description)/urdf/fishbot/common_inertia.xacro" />
     <!-- 相机传感器 -->
     <xacro:macro name="camera_xacro" params="xyz">
@@ -13,4 +14,14 @@
                 </material>
             </visual>
+            <collision>
+                <origin xyz="0 0 0" rpy="0 0 0" />
+                <geometry>
+                    <box size="0.02 0.01 0.02" />
+                </geometry>
+                <material name="green">
+                    <color rgba="0 1.0 0 0.8" />
+                </material>
+            </collision>
+            <xacro:box_inertia m="0.1" w="0.02" h="0.01" d="0.02" />
         </link>
         <joint name="camera_joint" type="fixed">

File: study/chapt6/chapt6_ws/src/fishbot_description/urdf/fishbot/sensor/imu.urdf.xacro (robot description, xacro)
@@ -1,4 +1,5 @@
 <?xml version="1.0"?>
 <robot xmlns:xacro="http://www.ros.org/wiki/xacro">
+    <xacro:include filename="$(find fishbot_description)/urdf/fishbot/common_inertia.xacro" />
     <!-- IMU传感器 -->
     <xacro:macro name="imu_xacro" params="xyz">
@@ -13,4 +14,14 @@
                 </material>
             </visual>
+            <collision>
+                <origin xyz="0 0 0" rpy="0 0 0"/>
+                <geometry>
+                    <box size="0.02 0.02 0.02" />
+                </geometry>
+                <material name="black">
+                    <color rgba="0 0 0.8" />
+                </material>
+            </collision>
+            <xacro:box_inertia m="0.05" w="0.02" h="0.02" d="0.02" />
         </link>
         <joint name="imu_joint" type="fixed">

File: study/chapt6/chapt6_ws/src/fishbot_description/urdf/fishbot/sensor/laser.urdf.xacro (robot description, xacro)
@@ -1,4 +1,6 @@
 <?xml version="1.0"?>
 <robot xmlns:xacro="http://www.ros.org/wiki/xacro">
+    <xacro:include filename="$(find fishbot_description)/urdf/fishbot/common_inertia.xacro" />
+    <!-- 激光雷达传感器 -->
     <xacro:macro name="laser_xacro" params="xyz">
         <link name="laser_cylinder_link">
@@ -12,4 +14,14 @@
                 </material>
             </visual>
+            <collision>
+                <origin xyz="0 0 0" rpy="0 0 0" />
+                <geometry>
+                    <cylinder length="0.1" radius="0.01" />
+                </geometry>
+                <material name="green">
+                    <color rgba="0 1.0 0 0.8" />
+                </material>
+            </collision>
+            <xacro:cylinder_inertia m="0.05" r="0.01" h="0.1" />
         </link>
         <joint name="laser_cylinder_joint" type="fixed">
@@ -28,4 +40,14 @@
                 </material>
             </visual>
+            <collision>
+                <origin xyz="0 0 0" rpy="0 0 0" />
+                <geometry>
+                    <cylinder length="0.02" radius="0.02" />
+                </geometry>
+                <material name="green">
+                    <color rgba="0 1.0 0 0.8" />
+                </material>
+            </collision>
+            <xacro:cylinder_inertia m="0.10" r="0.02" h="0.02" />
         </link>
         <joint name="laser_joint" type="fixed">
