Commit message: tbc

File: study/chapt6/chapt6_ws/src/fishbot_description/urdf/fishbot/actuator/caster.urdf.xacro (robot description, xacro)
@@ -23,5 +23,7 @@
                 </material>
             </collision>
-            <xacro:sphere_inertia m="0.05" r="0.016" />
+            <inertial>
+                <xacro:sphere_inertia m="0.05" r="0.016" />
+            </inertial>
         </link>
         <joint name="${caster_name}_caster_joint" type="fixed">

File: study/chapt6/chapt6_ws/src/fishbot_description/urdf/fishbot/actuator/wheel.urdf.xacro (robot description, xacro)
@@ -23,5 +23,7 @@
                 </material>
             </collision>
-            <xacro:cylinder_inertia m="0.05" r="0.032" h="0.04" />
+            <inertial>
+                <xacro:cylinder_inertia m="0.05" r="0.032" h="0.04" />
+            </inertial>
         </link>
         <joint name="${wheel_name}_wheel_joint" type="continuous">

File: study/chapt6/chapt6_ws/src/fishbot_description/urdf/fishbot/base.urdf.xacro (robot description, xacro)
@@ -5,10 +5,4 @@
     <!-- 机器人底座 -->
     <xacro:macro name="base_xacro" params="length radius">
-        <link name="base_footprint" />
-        <joint name="base_joint" type="fixed">
-            <parent link="base_footprint"/>
-            <child link="base_link"/>
-            <origin xyz="0 0 ${length/2.0+0.032-0.001}" rpy="0 0 0" />
-        </joint>
         <link name="base_link">
             <visual>
@@ -27,5 +21,7 @@
                 </geometry>
             </collision>
-            <xacro:cylinder_inertia m="1.0" r="${radius}" h="${length}" />
+            <inertial>
+                <xacro:cylinder_inertia m="1.0" r="${radius}" h="${length}" />
+            </inertial>
         </link>
     </xacro:macro>

File: study/chapt6/chapt6_ws/src/fishbot_description/urdf/fishbot/sensor/camera.urdf.xacro (robot description, xacro)
@@ -23,5 +23,7 @@
                 </material>
             </collision>
-            <xacro:box_inertia m="0.1" w="0.02" h="0.01" d="0.02" />
+            <inertial>
+                <xacro:box_inertia m="0.1" w="0.02" h="0.01" d="0.02" />
+            </inertial>
         </link>
         <joint name="camera_joint" type="fixed">

File: study/chapt6/chapt6_ws/src/fishbot_description/urdf/fishbot/sensor/imu.urdf.xacro (robot description, xacro)
@@ -23,5 +23,7 @@
                 </material>
             </collision>
-            <xacro:box_inertia m="0.05" w="0.02" h="0.02" d="0.02" />
+            <inertial>
+                <xacro:box_inertia m="0.05" w="0.02" h="0.02" d="0.02" />
+            </inertial>
         </link>
         <joint name="imu_joint" type="fixed">

File: study/chapt6/chapt6_ws/src/fishbot_description/urdf/fishbot/sensor/laser.urdf.xacro (robot description, xacro)
@@ -23,5 +23,7 @@
                 </material>
             </collision>
-            <xacro:cylinder_inertia m="0.05" r="0.01" h="0.1" />
+            <inertial>
+                <xacro:cylinder_inertia m="0.05" r="0.01" h="0.1" />
+            </inertial>
         </link>
         <joint name="laser_cylinder_joint" type="fixed">
@@ -49,5 +51,7 @@
                 </material>
             </collision>
-            <xacro:cylinder_inertia m="0.10" r="0.02" h="0.02" />
+            <inertial>
+                <xacro:cylinder_inertia m="0.10" r="0.02" h="0.02" />
+            </inertial>
         </link>
         <joint name="laser_joint" type="fixed">
