Commit message: 6.4.5 tbc

File: study/chapt6/chapt6_ws/src/fishbot_description/urdf/fishbot/actuator/wheel.urdf.xacro (robot description, xacro)
@@ -30,6 +30,8 @@
             <parent link="base_link"/>
             <child link="${wheel_name}_wheel_link"/>
-            <origin xyz="${xyz}" />
+            <origin xyz="${xyz}" rpy="0 0 0" />
             <axis xyz="0 1 0"/>
+            <limit effort="100" velocity="100" />
+            <dynamics damping="0.1" friction="0.1" />
         </joint>
     </xacro:macro>

File: study/chapt6/chapt6_ws/src/fishbot_description/urdf/fishbot/base.urdf.xacro (robot description, xacro)
@@ -5,4 +5,10 @@
     <!-- 机器人底座 -->
     <xacro:macro name="base_xacro" params="length radius">
+        <link name="base_footprint"/>
+        <joint name="base_link_joint" type="fixed">
+            <parent link="base_footprint"/>
+            <child link="base_link"/>
+            <origin xyz="0 0 ${length/2.0+0.032-0.001}" rpy="0 0 0"/>
+        </joint>
         <link name="base_link">
             <visual>

File: study/chapt6/chapt6_ws/src/fishbot_description/urdf/fishbot/fishbot.urdf.xacro (robot description, xacro)
@@ -10,4 +10,6 @@
     <xacro:include filename="$(find fishbot_description)/urdf/fishbot/actuator/wheel.urdf.xacro" />
     <xacro:include filename="$(find fishbot_description)/urdf/fishbot/actuator/caster.urdf.xacro" />
+    <!-- 包含gazebo插件宏定义 -->
+    <xacro:include filename="$(find fishbot_description)/urdf/fishbot/plugins/fishbot_gazebo.xacro" />
     <!-- 基座 -->
     <xacro:base_xacro length="0.12" radius="0.1" />
@@ -21,28 +23,3 @@
     <xacro:caster_xacro caster_name="front" xyz="0.08 0.0 -0.076" />
     <xacro:caster_xacro caster_name="back" xyz="-0.08 0.0 -0.076" />
-    <!-- ros2_control -->
-    <ros2_control name="FishbotController" type="system">
-        <hardware>
-            <plugin>gazebo_ros2_control/GazeboSystemPlugin</plugin>
-        </hardware>
-        <!-- 定义车轮关节的控制接口 -->
-        <joints>
-            <joint name="left_wheel_joint" />
-                <command_interface name="velocity" />
-                <state_interface name="position" />
-                <state_interface name="velocity" />
-            </joint>
-            <joint name="right_wheel_joint" />
-                <command_interface name="velocity" />
-                <state_interface name="position" />
-                <state_interface name="velocity" />
-            </joint>
-        </joints>
-    </ros2_control>
-    <!-- 为gazebo添加控制器插件 -->
-    <gazebo>
-        <plugin name="gazebo_ros2_control" filename="libgazebo_ros2_control.so">
-            <parameters>$(find fishbot_description)/config/controllers.yaml</parameters>
-        </plugin>
-    </gazebo>
 </robot>
