Commit message: lidar simulate done

File: study/chapt6/chapt6_ws/src/fishbot_description/urdf/fishbot/sensor/laser.urdf.xacro (robot description, xacro)
@@ -4,60 +4,84 @@
     <!-- 激光雷达传感器 -->
     <xacro:macro name="laser_xacro" params="xyz">
+        <!-- 雷达支撑柱 -->
         <link name="laser_cylinder_link">
             <visual>
-                <origin xyz="0 0 0" rpy="0 0 0" />
+                <origin xyz="0 0 0" rpy="0 0 0"/>
                 <geometry>
-                    <cylinder length="0.1" radius="0.01" />
+                    <cylinder length="0.1" radius="0.01"/>
                 </geometry>
                 <material name="green">
-                    <color rgba="0 1.0 0 0.8" />
+                    <color rgba="0 1.0 0 0.8"/>
                 </material>
             </visual>
             <collision>
-                <origin xyz="0 0 0" rpy="0 0 0" />
+                <origin xyz="0 0 0" rpy="0 0 0"/>
                 <geometry>
-                    <cylinder length="0.1" radius="0.01" />
+                    <cylinder length="0.1" radius="0.01"/>
                 </geometry>
-                <material name="green">
-                    <color rgba="0 1.0 0 0.8" />
-                </material>
             </collision>
             <inertial>
-                <xacro:cylinder_inertia m="0.05" r="0.01" h="0.1" />
+                <xacro:cylinder_inertia m="0.05" r="0.01" h="0.1"/>
             </inertial>
         </link>
         <joint name="laser_cylinder_joint" type="fixed">
-            <parent link="base_link" />
-            <child link="laser_cylinder_link" />
-            <origin xyz="${xyz}" />
+            <parent link="base_link"/>
+            <child link="laser_cylinder_link"/>
+            <origin xyz="${xyz}"/>
         </joint>
+        <!-- 雷达主体 -->
         <link name="laser_link">
             <visual>
-                <origin xyz="0 0 0" rpy="0 0 0" />
+                <origin xyz="0 0 0" rpy="0 0 0"/>
                 <geometry>
-                    <cylinder length="0.02" radius="0.02" />
+                    <cylinder length="0.02" radius="0.02"/>
                 </geometry>
                 <material name="green">
-                    <color rgba="0 1.0 0 0.8" />
+                    <color rgba="0 1.0 0 0.8"/>
                 </material>
             </visual>
             <collision>
-                <origin xyz="0 0 0" rpy="0 0 0" />
+                <origin xyz="0 0 0" rpy="0 0 0"/>
                 <geometry>
-                    <cylinder length="0.02" radius="0.02" />
+                    <cylinder length="0.02" radius="0.02"/>
                 </geometry>
-                <material name="green">
-                    <color rgba="0 1.0 0 0.8" />
-                </material>
             </collision>
             <inertial>
-                <xacro:cylinder_inertia m="0.10" r="0.02" h="0.02" />
+                <xacro:cylinder_inertia m="0.10" r="0.02" h="0.02"/>
             </inertial>
         </link>
         <joint name="laser_joint" type="fixed">
-            <parent link="laser_cylinder_link" />
-            <child link="laser_link" />
-            <origin xyz="0 0 0.05" />
+            <parent link="laser_cylinder_link"/>
+            <child link="laser_link"/>
+            <origin xyz="0 0 0.05"/>
         </joint>
+        <!-- Ignition Gazebo 激光雷达插件 -->
+        <gazebo reference="laser_link">
+            <sensor name="lidar" type="gpu_lidar">
+                <!-- <optical_frame_id>laser_link</optical_frame_id> -->
+                <update_rate>20</update_rate>
+                <topic>scan_raw</topic>
+                <ray>
+                    <scan>
+                        <horizontal>
+                            <samples>720</samples>
+                            <resolution>1</resolution>
+                            <min_angle>-3.14159</min_angle>
+                            <max_angle>3.14159</max_angle>
+                        </horizontal>
+                    </scan>
+                    <range>
+                        <min>0.12</min>
+                        <max>12.0</max>
+                        <resolution>0.01</resolution>
+                    </range>
+                    <noise>
+                        <type>gaussian</type>
+                        <mean>0.0</mean>
+                        <stddev>0.01</stddev>
+                    </noise>
+                </ray>
+            </sensor>
+        </gazebo>
     </xacro:macro>
 </robot>
