Commit message: 7.4 tbd : )

File: study/chapt6/chapt6_ws/src/fishbot_description/urdf/fishbot/ros2_control/mobile_base.ros2_control.xacro (robot description, xacro)
@@ -1,5 +1,4 @@
-<?xml version="1.0"?>
+<!-- <?xml version="1.0"?>
 <robot xmlns:xacro="http://www.ros.org/wiki/xacro">
-    <!--  ROS2 Control -->
     <ros2_control name="MobileBaseHardwareInterface" type="system">
         <hardware>
@@ -18,3 +17,28 @@
         </joint>
     </ros2_control>
+</robot> -->
+<?xml version="1.0"?>
+<robot xmlns:xacro="http://www.ros.org/wiki/xacro">
+    <ros2_control name="MG6010System" type="system">
+      <hardware>
+        <plugin>mg6010_can_control/MG6010System</plugin>
+        <param name="can_interface">can0</param>
+        <param name="bitrate">1000000</param>
+      </hardware>
+      <joint name="left_wheel_joint">
+        <command_interface name="velocity"/>
+        <state_interface   name="position"/>
+        <state_interface   name="velocity"/>
+        <state_interface   name="effort"/>
+        <param name="id">1</param>
+      </joint>
+      <joint name="right_wheel_joint">
+        <command_interface name="velocity"/>
+        <state_interface   name="position"/>
+        <state_interface   name="velocity"/>
+        <state_interface   name="effort"/>
+        <param name="id">2</param>
+      </joint>
+    </ros2_control>
+  </xacro:macro>
 </robot>
